File: riley-penny-custom.kicad_sch (KiCad schematic)
At the start: 12 parts, among them J1 Barrel_Jack_Switch, J2 AudioJack_TRS, J3 AudioJack_TRS, J4 Conn_01x08, J5 Conn_01x08, Q1 Q_PMOS_GSD

Commit message: finished schematics, started PCB
Parts:
- removed J4, J5: Conn_01x08, symbol Connector_Generic:Conn_01x08
- added J4, J5: Conn_01x06, bca-footprints:Pin_Header_Straight_1x06_Pitch2.54mm, symbol Connector_Generic:Conn_01x06
- added R2, R3: 22k, Resistor_SMD:R_0805_2012Metric_Pad1.20x1.40mm_HandSolder, symbol bca-symbols:R
Connections:
- net +9V: now also R2.2, R3.2
- net Earth: now also J4.1 (Pin_1), J5.1 (Pin_1)
- net bluesdriver-return: now also J5.4 (Pin_4)
- net bluesdriver-send: now also J5.3 (Pin_3)
- net input_jack: now also J4.2 (Pin_2)
- net output_jack: now also J5.5 (Pin_5)
- net zendrive_return: now also J4.4 (Pin_4)
- net zendrive_send: now also J4.3 (Pin_3)
- new net V+0: J4.6 (Pin_6), R2.1
- new net V+1: J5.6 (Pin_6), R3.1
Other:
- moved on the sheet: C1, C2, D1, FB1, G1, J1, J2, J3, Q1, R1
